Commit message: ros control in gazebo works

File: src/baldybot_bringup/description/ros2_control.xacro (robot description, xacro)
@@ -38,5 +38,5 @@
                 <plugin>gazebo_ros2_control/GazeboSystem</plugin>
             </hardware>
-            <joint name="right_front_wheel_joint">
+            <joint name="base_right_front_wheel_joint">
                 <command_interface name="velocity">
                     <param name="min">-10</param>
@@ -46,13 +46,5 @@
                 <state_interface name="position"/>
             </joint>
-            <!-- <joint name="right_back_wheel_joint">
-                <command_interface name="velocity">
-                    <param name="min">-10</param>
-                    <param name="max">10</param>
-                </command_interface>
-                <state_interface name="velocity"/>
-                <state_interface name="position"/>
-            </joint> -->
-            <joint name="left_front_wheel_joint">
+            <joint name="base_right_back_wheel_joint">
                 <command_interface name="velocity">
                     <param name="min">-10</param>
@@ -62,5 +54,5 @@
                 <state_interface name="position"/>
             </joint>
-            <!-- <joint name="left_back_wheel_joint">
+            <joint name="base_left_front_wheel_joint">
                 <command_interface name="velocity">
                     <param name="min">-10</param>
@@ -69,5 +61,13 @@
                 <state_interface name="velocity"/>
                 <state_interface name="position"/>
-            </joint> -->
+            </joint>
+            <joint name="base_left_back_wheel_joint">
+                <command_interface name="velocity">
+                    <param name="min">-10</param>
+                    <param name="max">10</param>
+                </command_interface>
+                <state_interface name="velocity"/>
+                <state_interface name="position"/>
+            </joint>
         </ros2_control>
      </xacro:if>
